File: Hardware/LC-Mainboard/LC-Mainboard.kicad_sch (KiCad schematic)
At the start: 43 parts, among them J1 Raspberry_Pi, J2 Charge Controller, U1 MAX3232IDW

Commit message: Do a little math
Co-Authored by: Libidja
Parts:
- J10: value (none) -> Port Enc.; footprint (none) -> Connector_JST:JST_XH_S4B-XH-A_1x04_P2.50mm_Horizontal
- J3: value (none) -> I²C; footprint (none) -> Connector_JST:JST_XH_S4B-XH-A_1x04_P2.50mm_Horizontal
- J4: value (none) -> Beacon; footprint (none) -> Connector_JST:JST_XH_S2B-XH-A_1x02_P2.50mm_Horizontal
- J5: value (none) -> Star.Motor; footprint (none) -> Connector_JST:JST_XH_S3B-XH-A_1x03_P2.50mm_Horizontal
- J6: value (none) -> Port Motor; footprint (none) -> Connector_JST:JST_XH_S3B-XH-A_1x03_P2.50mm_Horizontal
- J7: value (none) -> DC In; footprint (none) -> Connector_JST:JST_XH_S3B-XH-A_1x03_P2.50mm_Horizontal
- J8: value (none) -> PTT; footprint (none) -> Connector_JST:JST_XH_S2B-XH-A_1x02_P2.50mm_Horizontal
- J9: value (none) -> Star.Enc.; footprint (none) -> Connector_JST:JST_XH_S4B-XH-A_1x04_P2.50mm_Horizontal
- R1, R2, R5, R6, R7, R9: value 100k -> (none)
- R3, R4, R8: value math -> (none)
Other:
- note added: "Check math with dad!"
Changed lines of the file:
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@@
+    (effects (font (size 1.27 1.27)) (justify left bottom))
+  )
+  (text "Check math with dad!" (at 205.105 43.18 0)
     (effects (font (size 1.27 1.27)) (justify left bottom))
   )
@@
       (effects (font (size 1.27 1.27)) (justify left))
     )
-    (property "Value" "100k" (id 1) (at 196.215 24.13 0)
+    (property "Value" "" (id 1) (at 196.215 24.13 0)
       (effects (font (size 1.27 1.27)) (justify left))
     )
@@
       (effects (font (size 1.27 1.27)) (justify left))
     )
-    (property "Value" "100k" (id 1) (at 178.435 24.13 0)
+    (property "Value" "" (id 1) (at 178.435 24.13 0)
       (effects (font (size 1.27 1.27)) (justify left))
     )
@@
     (in_bom yes) (on_board yes)
     (property "Reference" "J3" (id 0) (at 22.225 21.59 0))
-    (property "Value" "" (id 1) (at 21.59 32.385 0))
-    (property "Footprint" "" (id 2) (at 21.59 25.4 0)
+    (property "Value" "I²C" (id 1) (at 21.59 32.385 0))
+    (property "Footprint" "Connector_JST:JST_XH_S4B-XH-A_1x04_P2.50mm_Horizontal" (id 2) (at 21.59 25.4 0)
       (effects (font (size 1.27 1.27)) hide)
     )
@@
     (in_bom yes) (on_board yes)
     (property "Reference" "J5" (id 0) (at 22.225 47.625 0))
-    (property "Value" "" (id 1) (at 21.59 55.88 0))
-    (property "Footprint" "" (id 2) (at 21.59 51.435 0)
+    (property "Value" "Star.Motor" (id 1) (at 21.59 55.88 0))
+    (property "Footprint" "Connector_JST:JST_XH_S3B-XH-A_1x03_P2.50mm_Horizontal" (id 2) (at 21.59 51.435 0)
       (effects (font (size 1.27 1.27)) hide)
     )
@@
     (in_bom yes) (on_board yes)
     (property "Reference" "J8" (id 0) (at 22.225 113.665 0))
-    (property "Value" "" (id 1) (at 22.225 118.745 0))
-    (property "Footprint" "" (id 2) (at 21.59 114.935 0)
+    (property "Value" "PTT" (id 1) (at 22.225 118.745 0))
+    (property "Footprint" "Connector_JST:JST_XH_S2B-XH-A_1x02_P2.50mm_Horizontal" (id 2) (at 21.59 114.935 0)
       (effects (font (size 1.27 1.27)) hide)
     )
@@
     (in_bom yes) (on_board yes)
     (property "Reference" "J10" (id 0) (at 22.225 86.995 0))
-    (property "Value" "" (id 1) (at 21.59 97.155 0))
-    (property "Footprint" "" (id 2) (at 21.59 90.805 0)
+    (property "Value" "Port Enc." (id 1) (at 21.59 97.155 0))
+    (property "Footprint" "Connector_JST:JST_XH_S4B-XH-A_1x04_P2.50mm_Horizontal" (id 2) (at 21.59 90.805 0)
       (effects (font (size 1.27 1.27)) hide)
     )
@@
       (effects (font (size 1.27 1.27)) (justify left))
     )
-    (property "Value" "100k" (id 1) (at 229.87 24.13 0)
+    (property "Value" "" (id 1) (at 229.87 24.13 0)
       (effects (font (size 1.27 1.27)) (justify left))
     )
@@
       (effects (font (size 1.27 1.27)) (justify left))
     )
-    (property "Value" "math" (id 1) (at 213.995 24.13 0)
+    (property "Value" "" (id 1) (at 213.995 24.13 0)
       (effects (font (size 1.27 1.27)) (justify left))
     )
@@
     (in_bom yes) (on_board yes)
     (property "Reference" "J4" (id 0) (at 22.225 37.465 0))
-    (property "Value" "" (id 1) (at 21.59 42.545 0))
-    (property "Footprint" "" (id 2) (at 21.59 38.735 0)
+    (property "Value" "Beacon" (id 1) (at 21.59 42.545 0))
+    (property "Footprint" "Connector_JST:JST_XH_S2B-XH-A_1x02_P2.50mm_Horizontal" (id 2) (at 21.59 38.735 0)
       (effects (font (size 1.27 1.27)) hide)
     )
@@
       (effects (font (size 1.27 1.27)) (justify left))
     )
-    (property "Value" "math" (id 1) (at 222.25 24.13 0)
+    (property "Value" "" (id 1) (at 222.25 24.13 0)
       (effects (font (size 1.27 1.27)) (justify left))
     )
@@
     (in_bom yes) (on_board yes)
     (property "Reference" "J6" (id 0) (at 22.225 74.93 0))
-    (property "Value" "" (id 1) (at 21.59 83.185 0))
-    (property "Footprint" "" (id 2) (at 21.59 78.74 0)
+    (property "Value" "Port Motor" (id 1) (at 21.59 83.185 0))
+    (property "Footprint" "Connector_JST:JST_XH_S3B-XH-A_1x03_P2.50mm_Horizontal" (id 2) (at 21.59 78.74 0)
       (effects (font (size 1.27 1.27)) hide)
     )
@@
       (effects (font (size 1.27 1.27)) (justify left))
     )
-    (property "Value" "math" (id 1) (at 205.105 24.13 0)
+    (property "Value" "" (id 1) (at 205.105 24.13 0)
       (effects (font (size 1.27 1.27)) (justify left))
     )
@@
       (effects (font (size 1.27 1.27)) (justify left))
     )
-    (property "Value" "100k" (id 1) (at 238.125 24.13 0)
+    (property "Value" "" (id 1) (at 238.125 24.13 0)
       (effects (font (size 1.27 1.27)) (justify left))
     )
@@
     (in_bom yes) (on_board yes)
     (property "Reference" "J7" (id 0) (at 22.225 101.6 0))
-    (property "Value" "" (id 1) (at 21.59 109.855 0))
-    (property "Footprint" "" (id 2) (at 21.59 105.41 0)
+    (property "Value" "DC In" (id 1) (at 21.59 109.855 0))
+    (property "Footprint" "Connector_JST:JST_XH_S3B-XH-A_1x03_P2.50mm_Horizontal" (id 2) (at 21.59 105.41 0)
       (effects (font (size 1.27 1.27)) hide)
     )
@@
     (in_bom yes) (on_board yes)
     (property "Reference" "J9" (id 0) (at 22.225 60.325 0))
-    (property "Value" "" (id 1) (at 21.59 70.485 0))
-    (property "Footprint" "" (id 2) (at 21.59 64.135 0)
+    (property "Value" "Star.Enc." (id 1) (at 21.59 70.485 0))
+    (property "Footprint" "Connector_JST:JST_XH_S4B-XH-A_1x04_P2.50mm_Horizontal" (id 2) (at 21.59 64.135 0)
       (effects (font (size 1.27 1.27)) hide)
     )
@@
       (effects (font (size 1.27 1.27)) (justify left))
     )
-    (property "Value" "100k" (id 1) (at 249.555 24.13 0)
+    (property "Value" "" (id 1) (at 249.555 24.13 0)
       (effects (font (size 1.27 1.27)) (justify left))
     )
@@
       (effects (font (size 1.27 1.27)) (justify left))
     )
-    (property "Value" "100k" (id 1) (at 187.325 24.13 0)
+    (property "Value" "" (id 1) (at 187.325 24.13 0)
       (effects (font (size 1.27 1.27)) (justify left))
     )
@@
     )
     (path "/c42da64f-4f91-4719-bb15-e561fd75de17"
-      (reference "R1") (unit 1) (value "100k") (footprint "Resistor_SMD:R_0805_2012Metric")
+      (reference "R1") (unit 1) (value "100R") (footprint "Resistor_SMD:R_0805_2012Metric")
     )
     (path "/e842b4d3-05c5-4fd1-8d89-8e0e8bfbdbba"
-      (reference "R2") (unit 1) (value "100k") (footprint "Resistor_SMD:R_0805_2012Metric")
+      (reference "R2") (unit 1) (value "100R") (footprint "Resistor_SMD:R_0805_2012Metric")
     )
     (path "/75bade5e-a47a-483f-8e61-60557be59a7d"
-      (reference "R3") (unit 1) (value "math") (footprint "Resistor_SMD:R_0805_2012Metric")
+      (reference "R3") (unit 1) (value "700R") (footprint "Resistor_SMD:R_0805_2012Metric")
     )
     (path "/aa4833b5-9f58-4ed3-b13c-70c3cdb83bb7"
-      (reference "R4") (unit 1) (value "math") (footprint "Resistor_SMD:R_0805_2012Metric")
+      (reference "R4") (unit 1) (value "220R") (footprint "Resistor_SMD:R_0805_2012Metric")
     )
     (path "/6f012ed3-15c4-489a-b433-26c0f45da341"
-      (reference "R5") (unit 1) (value "100k") (footprint "Resistor_SMD:R_0805_2012Metric")
+      (reference "R5") (unit 1) (value "100R") (footprint "Resistor_SMD:R_0805_2012Metric")
     )
     (path "/1c8d1cca-fb11-47a7-855f-9a1005464a84"
-      (reference "R6") (unit 1) (value "100k") (footprint "Resistor_SMD:R_0805_2012Metric")
+      (reference "R6") (unit 1) (value "100R") (footprint "Resistor_SMD:R_0805_2012Metric")
     )
     (path "/1e305f30-3580-41a5-a110-ca02a46cb34f"
-      (reference "R7") (unit 1) (value "100k") (footprint "Resistor_SMD:R_0805_2012Metric")
+      (reference "R7") (unit 1) (value "100R") (footprint "Resistor_SMD:R_0805_2012Metric")
     )
     (path "/bc610b4b-4822-4a8a-b60a-14fc9fe5f094"
-      (reference "R8") (unit 1) (value "math") (footprint "Resistor_SMD:R_0805_2012Metric")
+      (reference "R8") (unit 1) (value "750R") (footprint "Resistor_SMD:R_0805_2012Metric")
     )
     (path "/eaf0b044-60de-4f40-9968-38e000e4b494"
-      (reference "R9") (unit 1) (value "100k") (footprint "Resistor_SMD:R_0805_2012Metric")
+      (reference "R9") (unit 1) (value "100R") (footprint "Resistor_SMD:R_0805_2012Metric")
     )
     (path "/5643cc66-5524-4eca-9c29-7b06fd8f2ec4"

Commit message: Most of the routing is patched up, review with dad!
Parts:
- added C5, C6: (no value), symbol Device:C_Small
- added U2: (no value), symbol Regulator_Linear:NCP1117-12_SOT223
- C1, C2, C3, C4: value 0.1μf -> (none); footprint Capacitor_SMD:C_0805_2012Metric -> (none)
- D1: value SLR_RX -> (none); footprint LED_SMD:LED_0805_2012Metric -> (none)
- D2: value SLR_TX -> (none); footprint LED_SMD:LED_0805_2012Metric -> (none)
- D3: value 12v -> (none); footprint LED_SMD:LED_0805_2012Metric -> (none)
- D4: value 5v -> (none); footprint LED_SMD:LED_0805_2012Metric -> (none)
- D5: value 3.3v -> (none); footprint LED_SMD:LED_0805_2012Metric -> (none)
- D6: value DCD -> (none); footprint LED_SMD:LED_0805_2012Metric -> (none)
- D7: value STAT -> (none); footprint LED_SMD:LED_0805_2012Metric -> (none)
- D8: value BATT -> (none); footprint LED_SMD:LED_0805_2012Metric -> (none)
- D9: value TX -> (none); footprint LED_SMD:LED_0805_2012Metric -> (none)
- H1, H2, H3, H4: value PiMountingHole -> (none); footprint MountingHole:MountingHole_3mm -> (none)
- H5, H6, H7: value BrdMountingHole -> (none); footprint MountingHole:MountingHole_3mm -> (none)
- J1: value Raspberry_Pi -> (none); footprint Connector_PinSocket_2.54mm:PinSocket_2x20_P2.54mm_Vertical -> (none)
- J10: value Port Enc. -> (none); footprint Connector_JST:JST_XH_S4B-XH-A_1x04_P2.50mm_Horizontal -> (none)
- J2: value Charge Controller -> (none); footprint Connector_RJ:RJ12_Amphenol_54601 -> (none)
- J3: value I²C -> (none); footprint Connector_JST:JST_XH_S4B-XH-A_1x04_P2.50mm_Horizontal -> (none)
- J4: value Beacon -> (none); footprint Connector_JST:JST_XH_S2B-XH-A_1x02_P2.50mm_Horizontal -> (none)
- J5: value Star.Motor -> (none); footprint Connector_JST:JST_XH_S3B-XH-A_1x03_P2.50mm_Horizontal -> (none)
- J6: value Port Motor -> (none); footprint Connector_JST:JST_XH_S3B-XH-A_1x03_P2.50mm_Horizontal -> (none)
- J7: value DC In -> (none); footprint Connector_JST:JST_XH_S3B-XH-A_1x03_P2.50mm_Horizontal -> (none)
- J8: value PTT -> (none); footprint Connector_JST:JST_XH_S2B-XH-A_1x02_P2.50mm_Horizontal -> (none)
- J9: value Star.Enc. -> (none); footprint Connector_JST:JST_XH_S4B-XH-A_1x04_P2.50mm_Horizontal -> (none)
- JP1, JP2: value VRM_JP -> (none); footprint Jumper:SolderJumper-2_P1.3mm_Open_Pad1.0x1.5mm -> (none)
- R1, R2, R3, R4, R5, R6, R7, R8, R9: footprint Resistor_SMD:R_0805_2012Metric -> (none)
- R10: value math -> (none); footprint Resistor_SMD:R_0805_2012Metric -> (none)
- U1: value MAX3232IDW -> (none); footprint KenwoodFox:MAX3232IDW -> (none)
Connections:
- net TX_LED is gone; now on net PTT: D9.1 (K)
- net +12V: now also C5.1, U2.3 (VI)
- net +5V: now also C6.1, U2.2 (VO)
- net GND: now also C5.2, C6.2, U2.1 (GND)
Other:
- note added: "This chip may be fine for the pi3 (less than 1A) but the pi4 can use up to 2A"
