File: Hardware/LC-Mainboard/LC-Mainboard.kicad_pcb (KiCad board)
At the start: 2 copper layers, 88 x 67 mm, 55 parts, among them J1 Raspberry_Pi, J10 Port Enc., J2 Charge Controller, J3 I²C, J4 Beacon, J5 Star.Motor, J6 Port Motor, J7 DC In, J8 PTT, J9 Star.Enc.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

Commit message: fixup! Add last touches and fix all DRC
Parts:
- U1: value DW16 -> MAX3232IDW
- moved R10 1.35 mm to (115.3, 120.4)
- moved J8 1.10 mm to (117.8, 125.0)
- moved J7 1.00 mm to (144.5, 125.0)
Routing:
- net +12V: track 121.2 -> 120.2 mm
- net PTT: track 116.1 -> 116.7 mm
Changed lines of the file:
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@@
   (net 63 "Net-(Q1-Pad3)")
   (net 64 "Net-(Q2-Pad1)")
-  (net 65 "Net-(R12-Pad1)")
+  (net 65 "Net-(Q2-Pad3)")
   (footprint "Package_TO_SOT_SMD:SOT-23" (layer "F.Cu")
     (at 118.9 87.2 90)
@@
       (net 20 "GND") (pinfunction "E") (pintype "passive"))
     (pad "3" smd roundrect (at 0.9375 0 90) (size 1.475 0.6) (layers "F.Cu" "F.Paste" "F.Mask") (roundrect_rratio 0.25)
-      (net 65 "Net-(R12-Pad1)") (pinfunction "C") (pintype "passive"))
+      (net 65 "Net-(Q2-Pad3)") (pinfunction "C") (pintype "passive"))
     (model "${KICAD6_3DMODEL_DIR}/Package_TO_SOT_SMD.3dshapes/SOT-23.wrl"
       (offset (xyz 0 0 0))
@@
       (effects (font (size 1 1) (thickness 0.15)))
     )
-    (fp_text value "DW16" (at 0 -3.5) (layer "F.Fab")
+    (fp_text value "MAX3232IDW" (at 0 -3.5) (layer "F.Fab")
       (effects (font (size 1 1) (thickness 0.15)))
     )
@@
   )
   (footprint "Resistor_SMD:R_0805_2012Metric" (layer "F.Cu")
-    (at 115.25 121.75 -90)
+    (at 115.3 120.4 -90)
     (descr "Resistor SMD 0805 (2012 Metric), square (rectangular) end terminal, IPC_7351 nominal, (Body size source: IPC-SM-782 page 72, https://www.pcb-3d.com/wordpress/wp-content/uploads/ipc-sm-782a_amendment_1_and_2.pdf), generated with kicad-footprint-generator")
     (tags "resistor")
@@
     (fp_line (start 1 -0.625) (end 1 0.625) (layer "F.Fab") (width 0.1))
     (pad "1" smd roundrect (at -0.9125 0 90) (size 1.025 1.4) (layers "F.Cu" "F.Paste" "F.Mask") (roundrect_rratio 0.243902)
-      (net 65 "Net-(R12-Pad1)") (pintype "passive"))
+      (net 65 "Net-(Q2-Pad3)") (pintype "passive"))
     (pad "2" smd roundrect (at 0.9125 0 90) (size 1.025 1.4) (layers "F.Cu" "F.Paste" "F.Mask") (roundrect_rratio 0.243902)
       (net 62 "Net-(Q1-Pad1)") (pintype "passive"))
@@
     (at 183.25 80)
     (attr board_only exclude_from_pos_files exclude_from_bom)
-    (fp_text reference "G***" (at 0 0) (layer "F.SilkS")
+    (fp_text reference "G***" (at 0 0) (layer "F.Fab")
       (effects (font (size 1.524 1.524) (thickness 0.3)))
     )
@@
     (at 183.75 105.5)
     (attr board_only exclude_from_pos_files exclude_from_bom)
-    (fp_text reference "G***" (at 0 0) (layer "F.SilkS")
+    (fp_text reference "G***" (at 0 0) (layer "F.Fab")
       (effects (font (size 1.524 1.524) (thickness 0.3)))
     )
@@
   )
   (footprint "Connector_JST:JST_XH_S2B-XH-A_1x02_P2.50mm_Horizontal" (layer "B.Cu")
-    (at 117.75 126.05 180)
+    (at 117.75 124.95 180)
     (descr "JST XH series connector, S2B-XH-A (http://www.jst-mfg.com/product/pdf/eng/eXH.pdf), generated with kicad-footprint-generator")
     (tags "connector JST XH horizontal")
@@
   )
   (footprint "Connector_JST:JST_XH_S3B-XH-A_1x03_P2.50mm_Horizontal" (layer "B.Cu")
-    (at 144.5 126 180)
+    (at 144.5 125 180)
     (descr "JST XH series connector, S3B-XH-A (http://www.jst-mfg.com/product/pdf/eng/eXH.pdf), generated with kicad-footprint-generator")
     (tags "connector JST XH horizontal")
@@
     (effects (font (size 0.508 0.508) (thickness 0.127)) (justify mirror))
   )
-  (gr_text "BAT" (at 139.5 124.2) (layer "B.SilkS")
+  (gr_text "BAT" (at 139.5 123.2) (layer "B.SilkS")
     (effects (font (size 0.508 0.508) (thickness 0.127)) (justify mirror))
   )
@@
     (effects (font (size 0.508 0.508) (thickness 0.127)) (justify mirror))
   )
-  (gr_text "12V" (at 142.1 124.2) (layer "B.SilkS")
+  (gr_text "12V" (at 142.1 123.2) (layer "B.SilkS")
     (effects (font (size 0.508 0.508) (thickness 0.127)) (justify mirror))
   )
@@
   (segment (start 113.58 82.22) (end 109 82.22) (width 0.35) (layer "F.Cu") (net 2))
   (segment (start 117.25 78.55) (end 113.58 82.22) (width 0.35) (layer "F.Cu") (net 2))
+  (segment (start 107.634511 121.685489) (end 106.46 122.86) (width 0.35) (layer "F.Cu") (net 17))
+  (segment (start 111.1 111.2) (end 112.424511 112.524511) (width 0.35) (layer "F.Cu") (net 17))
+  (segment (start 112.424511 112.524511) (end 112.424511 116.875489) (width 0.35) (layer "F.Cu") (net 17))
+  (segment (start 108.513501 119.145489) (end 107.634511 120.024479) (width 0.35) (layer "F.Cu") (net 17))
   (segment (start 114.3875 88.2) (end 114.3875 90.3125) (width 0.35) (layer "F.Cu") (net 17))
-  (segment (start 110.154511 119.145489) (end 108.513501 119.145489) (width 0.35) (layer "F.Cu") (net 17))
   (segment (start 107.634511 120.024479) (end 107.634511 121.685489) (width 0.35) (layer "F.Cu") (net 17))
+  (segment (start 110.154511 119.145489) (end 108.513501 119.145489) (width 0.35) (layer "F.Cu") (net 17))
   (segment (start 114.3875 90.3125) (end 114.1 90.6) (width 0.35) (layer "F.Cu") (net 17))
-  (segment (start 108.513501 119.145489) (end 107.634511 120.024479) (width 0.35) (layer "F.Cu") (net 17))
   (segment (start 112.424511 116.875489) (end 110.154511 119.145489) (width 0.35) (layer "F.Cu") (net 17))
-  (segment (start 112.424511 112.324511) (end 112.424511 116.875489) (width 0.35) (layer "F.Cu") (net 17))
-  (segment (start 107.634511 121.685489) (end 106.46 122.86) (width 0.35) (layer "F.Cu") (net 17))
-  (segment (start 111.2 111.1) (end 112.424511 112.324511) (width 0.35) (layer "F.Cu") (net 17))
-  (via (at 111.2 111.1) (size 0.8) (drill 0.4) (layers "F.Cu" "B.Cu") (net 17))
+  (via (at 111.1 111.2) (size 0.8) (drill 0.4) (layers "F.Cu" "B.Cu") (net 17))
   (via (at 114.1 90.6) (size 0.8) (drill 0.4) (layers "F.Cu" "B.Cu") (net 17))
-  (segment (start 111.1 111.2) (end 111.2 111.1) (width 0.35) (layer "B.Cu") (net 17))
-  (segment (start 114.1 108.2) (end 111.2 111.1) (width 0.35) (layer "B.Cu") (net 17))
-  (segment (start 114.1 90.6) (end 114.1 108.2) (width 0.35) (layer "B.Cu") (net 17))
+  (segment (start 111.1 111.2) (end 114.1 108.2) (width 0.35) (layer "B.Cu") (net 17))
+  (segment (start 114.1 108.2) (end 114.1 90.6) (width 0.35) (layer "B.Cu") (net 17))
   (segment (start 119.765 99.135) (end 121.7 97.2) (width 0.35) (layer "F.Cu") (net 18))
   (segment (start 117.4788 99.135) (end 119.765 99.135) (width 0.35) (layer "F.Cu") (net 18))
@@
   (segment (start 134.3 93.2) (end 131.5 90.4) (width 0.7) (layer "F.Cu") (net 48))
   (segment (start 125.1 90.4) (end 122.9625 88.2625) (width 0.7) (layer "F.Cu") (net 48))
-  (segment (start 142 119.6375) (end 142 126) (width 0.7) (layer "F.Cu") (net 48))
-  (segment (start 122.9625 88.2625) (end 122.9625 84.35) (width 0.7) (layer "F.Cu") (net 48))
   (segment (start 141.3625 119) (end 142 119.6375) (width 0.7) (layer "F.Cu") (net 48))
+  (segment (start 142 119.6375) (end 142 125) (width 0.7) (layer "F.Cu") (net 48))
+  (segment (start 122.9625 88.2625) (end 122.9625 84.35) (width 0.7) (layer "F.Cu") (net 48))
   (segment (start 120.9 84.3125) (end 122.925 84.3125) (width 0.35) (layer "F.Cu") (net 48))
   (segment (start 126.5 90.4) (end 125.1 90.4) (width 0.7) (layer "F.Cu") (net 48))
@@
   (segment (start 139.5 126) (end 146.7 133.2) (width 0.35) (layer "F.Cu") (net 55))
   (segment (start 166.3 133.2) (end 179.9 119.6) (width 0.35) (layer "F.Cu") (net 55))
-  (segment (start 115.25 122.6625) (end 115.25 126.05) (width 0.35) (layer "F.Cu") (net 56))
-  (segment (start 115.2125 120.8) (end 115.25 120.8375) (width 0.35) (layer "F.Cu") (net 57))
-  (segment (start 113.1 121.6) (end 113.9 120.8) (width 0.35) (layer "F.Cu") (net 57))
-  (segment (start 113.9 120.8) (end 115.2125 120.8) (width 0.35) (layer "F.Cu") (net 57))
+  (segment (start 115.3 121.3125) (end 115.25 121.3625) (width 0.35) (layer "F.Cu") (net 56))
+  (segment (start 115.25 121.3625) (end 115.25 124.95) (width 0.35) (layer "F.Cu") (net 56))
+  (segment (start 113.1 129.4) (end 113.1 121.6875) (width 0.35) (layer "F.Cu") (net 57))
+  (segment (start 113.1 121.6875) (end 115.3 119.4875) (width 0.35) (layer "F.Cu") (net 57))
   (segment (start 168.7125 102.6) (end 169.8125 101.5) (width 0.35) (layer "F.Cu") (net 57))
   (segment (start 166.7 102.6) (end 168.7125 102.6) (width 0.35) (layer "F.Cu") (net 57))
-  (segment (start 113.1 129.4) (end 113.1 121.6) (width 0.35) (layer "F.Cu") (net 57))
   (via (at 166.7 102.6) (size 0.8) (drill 0.4) (layers "F.Cu" "B.Cu") (net 57))
   (via (at 113.1 129.4) (size 0.8) (drill 0.4) (layers "F.Cu" "B.Cu") (net 57))

Commit message: Change direction, pi can now control load control
Parts:
- added J11: Load En., Connector_JST:JST_XH_S2B-XH-A_1x02_P2.50mm_Horizontal, B.Cu at (135.3, 125.2)
- added Q3: MMBT3904, Package_TO_SOT_SMD:SOT-23, F.Cu at (122.5, 116.6)
- added R15: 1K, Resistor_SMD:R_0805_2012Metric, F.Cu at (119.5, 116.6)
- D3: value 12v -> BATT
- D8: value BATT -> LOAD
- J7: footprint Connector_JST:JST_XH_S3B-XH-A_1x03_P2.50mm_Horizontal -> Connector_JST:JST_XH_S2B-XH-A_1x02_P2.50mm_Horizontal
- moved J7 0.21 mm to (144.3, 125.2)
Connections:
- J1 pad 21: unconnected-(J1-Pad21) -> LOAD_EN_Pi
- R8 pad 1: +12VA -> LOAD_EN
Routing:
- net LOAD_EN: track 0.00 -> 115.9 mm
- net +12VA: track 91.6 -> 0.00 mm
- net LOAD_EN_Pi: track 0.00 -> 25.8 mm, vias 0 -> 2
- net +5V: track 149.9 -> 166.7 mm, vias 1 -> 3
- net GND: track 0.00 -> 6.13 mm, vias 16 -> 17
- net +3V3: track 156.9 -> 154.7 mm
- net Net-(Q3-Pad1): track 0.00 -> 2.08 mm
Other:
- board text added: "RELAY"
- board text removed: "12V"

Commit message: Its done, all systems checked and final
Parts:
- moved C5 0.80 mm to (143.1, 119.0)
Routing:
- net +12V: track 120.2 -> 121.0 mm
- net STAR_PWM: track 59.8 -> 59.1 mm
Changed lines of the file:
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@@
   )
   (footprint "Capacitor_SMD:C_Elec_6.3x5.4" (layer "F.Cu")
-    (at 143.9 119)
+    (at 143.1 119)
     (descr "SMD capacitor, aluminum electrolytic nonpolar, 6.3x5.4mm")
     (tags "capacitor electrolyic nonpolar")
@@
     (pad "6" thru_hole circle (at 6.35 -2.54 180) (size 1.52 1.52) (drill 0.76) (layers *.Cu *.Mask)
       (net 22 "unconnected-(J2-Pad6)") (pintype "passive+no_connect"))
-    (model "${KICAD6_3DMODEL_DIR}/Connector_RJ.3dshapes/RJ12_Amphenol_54601.wrl"
+    (model "${KENWOODFOX_3DMODELS}/RJ12.wrl"
       (offset (xyz 0 0 0))
       (scale (xyz 1 1 1))
@@
   (segment (start 128.4125 78.7125) (end 128.25 78.55) (width 0.7) (layer "F.Cu") (net 39))
   (segment (start 128.4125 83.4) (end 128.4125 78.7125) (width 0.7) (layer "F.Cu") (net 39))
-  (segment (start 132.5 119.4) (end 135.7 119.4) (width 0.35) (layer "F.Cu") (net 40))
-  (segment (start 132.3 119.2) (end 132.5 119.4) (width 0.35) (layer "F.Cu") (net 40))
-  (segment (start 135.7 119.4) (end 137.3 121) (width 0.35) (layer "F.Cu") (net 40))
+  (segment (start 132.5 119.4) (end 132.3 119.2) (width 0.35) (layer "F.Cu") (net 40))
+  (segment (start 136.7 119.4) (end 132.5 119.4) (width 0.35) (layer "F.Cu") (net 40))
+  (segment (start 137.5 120.2) (end 136.7 119.4) (width 0.35) (layer "F.Cu") (net 40))
   (via (at 132.3 119.2) (size 0.8) (drill 0.4) (layers "F.Cu" "B.Cu") (net 40))
-  (via (at 137.3 121) (size 0.8) (drill 0.4) (layers "F.Cu" "B.Cu") (net 40))
+  (via (at 137.5 120.2) (size 0.8) (drill 0.4) (layers "F.Cu" "B.Cu") (net 40))
   (segment (start 132.3 119.2) (end 131.7 119.8) (width 0.35) (layer "B.Cu") (net 40))
-  (segment (start 150.74952 113.49952) (end 144.80048 113.49952) (width 0.35) (layer "B.Cu") (net 40))
-  (segment (start 144.80048 113.49952) (end 137.3 121) (width 0.35) (layer "B.Cu") (net 40))
+  (segment (start 150.74952 113.49952) (end 160 122.75) (width 0.35) (layer "B.Cu") (net 40))
+  (segment (start 144.80048 113.49952) (end 150.74952 113.49952) (width 0.35) (layer "B.Cu") (net 40))
   (segment (start 131.7 119.8) (end 111.02 119.8) (width 0.35) (layer "B.Cu") (net 40))
-  (segment (start 160 122.75) (end 150.74952 113.49952) (width 0.35) (layer "B.Cu") (net 40))
+  (segment (start 137.5 120.2) (end 138.1 120.2) (width 0.35) (layer "B.Cu") (net 40))
+  (segment (start 138.1 120.2) (end 144.80048 113.49952) (width 0.35) (layer "B.Cu") (net 40))
   (segment (start 111.02 119.8) (end 109 117.78) (width 0.35) (layer "B.Cu") (net 40))
   (segment (start 126.11101 97.25) (end 109.36101 114) (width 0.35) (layer "B.Cu") (net 41))
@@
   (segment (start 134.3 98.6) (end 134.3 93.2) (width 0.7) (layer "F.Cu") (net 47))
   (segment (start 122.925 84.3125) (end 122.9625 84.35) (width 0.35) (layer "F.Cu") (net 47))
+  (segment (start 140.5625 119) (end 142 120.4375) (width 0.7) (layer "F.Cu") (net 47))
   (segment (start 141.5 108.6) (end 141.2 108.9) (width 0.7) (layer "F.Cu") (net 47))
   (segment (start 141.2 108.9) (end 141.2 112.95) (width 0.7) (layer "F.Cu") (net 47))
   (segment (start 175.1625 86.5) (end 175.1625 87.4625) (width 0.35) (layer "F.Cu") (net 47))
-  (segment (start 141.2 112.95) (end 141.2 118.8375) (width 0.7) (layer "F.Cu") (net 47))
   (segment (start 175.1625 87.4625) (end 175.7 88) (width 0.35) (layer "F.Cu") (net 47))
   (segment (start 134.3 93.2) (end 131.5 90.4) (width 0.7) (layer "F.Cu") (net 47))
   (segment (start 125.1 90.4) (end 122.9625 88.2625) (width 0.7) (layer "F.Cu") (net 47))
-  (segment (start 141.3625 119) (end 142 119.6375) (width 0.7) (layer "F.Cu") (net 47))
-  (segment (start 142 119.6375) (end 142 125) (width 0.7) (layer "F.Cu") (net 47))
+  (segment (start 141.2 112.95) (end 141.2 118.8375) (width 0.7) (layer "F.Cu") (net 47))
   (segment (start 122.9625 88.2625) (end 122.9625 84.35) (width 0.7) (layer "F.Cu") (net 47))
   (segment (start 120.9 84.3125) (end 122.925 84.3125) (width 0.35) (layer "F.Cu") (net 47))
+  (segment (start 141.0375 119) (end 140.5625 119) (width 0.7) (layer "F.Cu") (net 47))
   (segment (start 126.5 90.4) (end 125.1 90.4) (width 0.7) (layer "F.Cu") (net 47))
-  (segment (start 141.2 118.8375) (end 141.3625 119) (width 0.7) (layer "F.Cu") (net 47))
+  (segment (start 141.2 118.8375) (end 141.0375 119) (width 0.7) (layer "F.Cu") (net 47))
+  (segment (start 142 120.4375) (end 142 125) (width 0.7) (layer "F.Cu") (net 47))
   (via (at 175.7 88) (size 0.8) (drill 0.4) (layers "F.Cu" "B.Cu") (net 47))
   (via (at 134.3 98.6) (size 0.8) (drill 0.4) (layers "F.Cu" "B.Cu") (net 47))
