File: Hardware/Dev_Card/Dev_Card.kicad_pcb (KiCad board)
At the start: 2 copper layers, 75 x 116.7 mm, 52 parts, among them J1 CON1, J2 CON2, J3 CON3, U1 ProtoBoard, U2 CARD ?

Commit message: Few fixups on the dev card
Routing:
- net Net-(U2-I2C_SDA): track 2.54 -> 35.6 mm
- net Net-(U2-CARD_EN): track 2.54 -> 35.4 mm
- net Net-(U2-I2C_SCL): track 2.54 -> 30.1 mm
- net Net-(U2-CARD_EN2): track 2.54 -> 29.9 mm
- net Net-(U2-GPIO1): track 2.54 -> 29.7 mm
- net Net-(U2-CANL): track 2.54 -> 26.7 mm
- net Net-(U2-GPIO2): track 2.54 -> 26.4 mm
- net Net-(U2-CARD_EN3): track 2.54 -> 26.2 mm
- net Net-(U2-CARD_EN4): track 2.54 -> 24.3 mm
- net Net-(U2-CANH): track 2.54 -> 23.7 mm
- net Net-(U2-GPIO3): track 2.54 -> 23.4 mm
- net Net-(U2-CARD_SEL4): track 2.54 -> 15.6 mm
- net Net-(U2-CARD_SEL3): track 2.54 -> 14.9 mm
- net Net-(U2-UNUSED4): track 2.54 -> 14.5 mm
- net Net-(U2-CARD_SEL2): track 2.54 -> 14.5 mm
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
Commit message: Add a little more silk to the dev card
Other:
- board text added: "V+"
Changed lines of the file:
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@@
 		(layer "F.SilkS")
+	)
+	(gr_text "V+"
+		(at 13.5 -20.5 -270)
+		(layer "B.SilkS")
+		(effects
+			(font
+				(size 1.1 1.1)
+				(thickness 0.275)
+				(bold yes)
+			)
+			(justify left mirror)
+		)
 	)
 	(gr_text "GND"
@@
 		)
 	)
+	(gr_text "V+"
+		(at 13.5 -102 -270)
+		(layer "B.SilkS")
+		(effects
+			(font
+				(size 1.1 1.1)
+				(thickness 0.275)
+				(bold yes)
+			)
+			(justify right mirror)
+		)
+	)
 	(gr_text "3"
 		(at 7.5 -13.5 0)
@@
 		)
 	)
+	(gr_text "V+"
+		(at 13.5 -102 270)
+		(layer "F.SilkS")
+		(effects
+			(font
+				(size 1.1 1.1)
+				(thickness 0.275)
+				(bold yes)
+			)
+			(justify right)
+		)
+	)
 	(gr_text "12V"
 		(at -26.5 -105 0)
@@
 		)
 	)
+	(gr_text "V+"
+		(at 13.5 -20.5 270)
+		(layer "F.SilkS")
+		(effects
+			(font
+				(size 1.1 1.1)
+				(thickness 0.275)
+				(bold yes)
+			)
+			(justify left)
+		)
+	)

Commit message: Add even more silkscreen
Parts:
- added LOGO1: LOGO, KenwoodFox:ROBOTSTREAMER_LOGO, B.Cu at (-30.0, -65.8)
- added LOGO2: LOGO, KenwoodFox:KITSUNE_LOGO, B.Cu at (-30.0, -81.0)
- added LOGO3: OSHW-Logo2_14.6x12mm_SilkScreen, Symbol:OSHW-Logo2_14.6x12mm_SilkScreen, B.Cu at (-30.0, -96.2)
Other:
- board text added: "JLCJLCJLCJLC"
