File: Hardware/KIT_Controller/KIT_Controller.kicad_pcb (KiCad board)
At the start: 2 copper layers, 75 x 116.7 mm, 53 parts, among them J201 Micro_SD_Card_Det1, J202 USB_BOOT, J203 USBC, SW101 TM1000, U101 Nokia_5110_LCD, U102 CARD ?, U202 W25Q128JVS, U203 NCP1117-3.3_SOT223, U205 RP2040, U301 CC1101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

Commit message: Pivot to feather design
Parts:
- removed C101: 4.7uf, Capacitor_SMD:C_0805_2012Metric
- removed JP101: SolderJumper_2_Bridged, Jumper:SolderJumper-2_P1.3mm_Bridged_Pad1.0x1.5mm
- removed SW101: TM1000, KenwoodFox:TM1000
- removed U101: Nokia_5110_LCD, Nokia_5110-3310_LCD:Nokia_5110-3310_LCD
- added A1: Adafruit_Feather_Generic, Module:Adafruit_Feather, F.Cu at (-27.8, -102.9)
- moved C217 212.1 mm to (33.5, -91.5)
- moved D101 212.1 mm to (8.29, -4.75)
- moved D103 212.1 mm to (8.29, -42.2)
- moved D104 212.1 mm to (-4.66, -4.75)
- moved H101 212.1 mm to (28.0, -11.5)
- moved H102 212.1 mm to (-30.0, -12.0)
- moved J201 212.1 mm to (21.5, -103.4)
- moved R208 212.1 mm to (29.1, -91.5)
- moved R209 212.1 mm to (29.1, -88.6)
- moved R210 212.1 mm to (29.1, -85.6)
- moved R215 212.1 mm to (31.0, -95.6)
- moved R216 212.1 mm to (31.0, -98.5)
- moved R217 212.1 mm to (31.0, -101.5)
- moved U102 212.1 mm to (0.00, 0.00)
- moved U301 212.1 mm to (26.5, -43.1)
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Connections:
- U102 pad 11: /SCL -> unconnected-(U102-I2C_SCL-Pad11)
- U102 pad 13: /SDA -> unconnected-(U102-I2C_SDA-Pad13)

Commit message: So near to a backplane prototype now
Parts:
- A1: moved to B.Cu
- moved A1 20.1 mm to (-7.70, -102.8), turned to 180 degrees

Commit message: New branch for next board
Parts:
- removed C201, C202: 27p, Capacitor_SMD:C_0805_2012Metric
- removed C203, C205: 10u, Capacitor_SMD:C_0805_2012Metric
- removed C204, C207, C208, C209, C210, C211, C212, C213, C214, C215: 100n, Capacitor_SMD:C_0805_2012Metric
- removed C206, C216: 1u, Capacitor_SMD:C_0805_2012Metric
- removed D102: BL2, LED_SMD:LED_0805_2012Metric
- removed J202: USB_BOOT, Connector_PinHeader_2.54mm:PinHeader_1x02_P2.54mm_Vertical
- removed J203: USBC, Connector_USB:USB_C_Receptacle_XKB_U262-16XN-4BVC11
- removed R101, R102, R103, R104: 450, Resistor_SMD:R_0805_2012Metric
- removed R201, R203: 1k, Resistor_SMD:R_0805_2012Metric
- removed R202: DNP, Resistor_SMD:R_0805_2012Metric
- removed R204, R205: 27, Resistor_SMD:R_0805_2012Metric
- removed R206, R207: 5K1, Resistor_SMD:R_0805_2012Metric
- removed U202: W25Q128JVS, Package_SO:SOIC-8_5.23x5.23mm_P1.27mm
- removed U203: NCP1117-3.3_SOT223, Package_TO_SOT_SMD:SOT-223-3_TabPin2
- removed U205: RP2040, Package_DFN_QFN:QFN-56-1EP_7x7mm_P0.4mm_EP3.2x3.2mm_ThermalVias
- removed Y201: Crystal, Crystal:Crystal_SMD_HC49-SD
- added J1: CAN, Connector_Wire:SolderWire-0.5sqmm_1x03_P4.6mm_D0.9mm_OD2.1mm_Relief, B.Cu at (19.4, -18.1)
Connections:
- A1 pad 2: unconnected-(A1-3V3-Pad2) -> +3V3
- A1 pad 4: unconnected-(A1-GND-Pad4) -> GND
- U102 pad 27: unconnected-(U102-CANH-Pad27) -> /CANH
- U102 pad 28: unconnected-(U102-CANL-Pad28) -> /CANL

Commit message: Bump pcb and can_controller
Parts:
- added C201: 27p, Capacitor_SMD:C_0805_2012Metric, F.Cu at (63.7, -80.3)
- added C202: 27p, Capacitor_SMD:C_0805_2012Metric, F.Cu at (63.7, -77.3)
- added C203: 10u, Capacitor_SMD:C_0805_2012Metric, F.Cu at (63.7, -74.3)
- added C204: 100n, Capacitor_SMD:C_0805_2012Metric, F.Cu at (63.7, -71.3)
- added C205: 10u, Capacitor_SMD:C_0805_2012Metric, F.Cu at (68.1, -80.3)
- added C206: 1u, Capacitor_SMD:C_0805_2012Metric, F.Cu at (68.1, -77.3)
- added C207: 100n, Capacitor_SMD:C_0805_2012Metric, F.Cu at (68.1, -74.3)
- added C208: 100n, Capacitor_SMD:C_0805_2012Metric, F.Cu at (68.1, -71.3)
- added C209: 100n, Capacitor_SMD:C_0805_2012Metric, F.Cu at (72.6, -80.3)
- added C210: 100n, Capacitor_SMD:C_0805_2012Metric, F.Cu at (72.6, -77.3)
- added C211: 100n, Capacitor_SMD:C_0805_2012Metric, F.Cu at (72.6, -74.3)
- added C212: 100n, Capacitor_SMD:C_0805_2012Metric, F.Cu at (72.6, -71.3)
- added C213: 100n, Capacitor_SMD:C_0805_2012Metric, F.Cu at (77.0, -80.3)
- added C214: 100n, Capacitor_SMD:C_0805_2012Metric, F.Cu at (77.0, -77.3)
- added C215: 100n, Capacitor_SMD:C_0805_2012Metric, F.Cu at (77.0, -74.3)
- added C216: 1u, Capacitor_SMD:C_0805_2012Metric, F.Cu at (77.0, -71.3)
- added D102: BL2, LED_SMD:LED_0805_2012Metric, F.Cu at (99.6, -72.3)
- added J202: USB_BOOT, Connector_PinHeader_2.54mm:PinHeader_1x02_P2.54mm_Vertical, F.Cu at (63.8, -54.5)
- added J203: USBC, Connector_USB:USB_C_Receptacle_XKB_U262-16XN-4BVC11, F.Cu at (85.1, -76.6)
- added R101: 450, Resistor_SMD:R_0805_2012Metric, F.Cu at (95.2, -80.4)
- added R102: 450, Resistor_SMD:R_0805_2012Metric, F.Cu at (95.2, -77.4)
- added R103: 450, Resistor_SMD:R_0805_2012Metric, F.Cu at (95.2, -74.5)
- added R104: 450, Resistor_SMD:R_0805_2012Metric, F.Cu at (95.2, -71.5)
- added R201: 1k, Resistor_SMD:R_0805_2012Metric, F.Cu at (78.3, -68.3)
- added R202: DNP, Resistor_SMD:R_0805_2012Metric, F.Cu at (78.3, -65.4)
- added R203: 1k, Resistor_SMD:R_0805_2012Metric, F.Cu at (78.3, -62.4)
- added R204: 27, Resistor_SMD:R_0805_2012Metric, F.Cu at (78.3, -59.5)
- added R205: 27, Resistor_SMD:R_0805_2012Metric, F.Cu at (78.3, -56.5)
- added R206: 5K1, Resistor_SMD:R_0805_2012Metric, F.Cu at (78.3, -53.6)
- added R207: 5K1, Resistor_SMD:R_0805_2012Metric, F.Cu at (78.3, -50.6)
- added U1: TXB0108PW, Package_SO:TSSOP-20_4.4x6.5mm_P0.65mm, F.Cu at (-5.64, -22.9)
- added U202: W25Q128JVS, Package_SO:SOIC-8_5.23x5.23mm_P1.27mm, F.Cu at (66.6, -60.2)
- added U203: NCP1117-3.3_SOT223, Package_TO_SOT_SMD:SOT-223-3_TabPin2, F.Cu at (85.4, -56.3)
- added U205: RP2040, Package_DFN_QFN:QFN-56-1EP_7x7mm_P0.4mm_EP3.2x3.2mm_ThermalVias, F.Cu at (85.2, -65.2)
- added Y201: Crystal, Crystal:Crystal_SMD_HC49-SD, F.Cu at (68.8, -66.7)
