File: Hardware/KIT_Controller/KIT_Controller.kicad_sch (KiCad schematic)
At the start: 15 parts, among them SW101 TM1000, U101 Nokia_5110_LCD, U102 CARD ?

Commit message: v1.1 Prototype (#11)
Parts:
- removed C101: 4.7uf, Capacitor_SMD:C_0805_2012Metric, symbol Device:C_Small
- removed JP101: SolderJumper_2_Bridged, Jumper:SolderJumper-2_P1.3mm_Bridged_Pad1.0x1.5mm, symbol Jumper:SolderJumper_2_Bridged
- removed SW101: TM1000, KenwoodFox:TM1000, symbol KenwoodFox:TM1000
- removed U101: Nokia_5110_LCD, Nokia_5110-3310_LCD:Nokia_5110-3310_LCD, symbol nokia_5110-3310_lcd:Nokia_5110_LCD
- added A1: Adafruit_Feather_Generic, Module:Adafruit_Feather, symbol MCU_Module:Adafruit_Feather_Generic
Connections:
- no-connect marks 8 -> 3

Commit message: New branch for next board
Parts:
- added J1: CAN, Connector_Wire:SolderWire-0.5sqmm_1x03_P4.6mm_D0.9mm_OD2.1mm_Relief, symbol Connector:Conn_01x03_Socket
Connections:
- net +3V3: now also A1.2 (3V3)
- net GND: now also A1.4 (GND), J1.2 (Pin_2)
- net CANH: now reaches U102.27 (CANH)
- net CANH: now also J1.3 (Pin_3)
- net CANL: now reaches U102.28 (CANL)
- net CANL: now also J1.1 (Pin_1)
- no-connect marks 3 -> 5
Other:
- moved on the sheet: A1, D101, D102, D103, D104, R101, R102, R103, R104, U102

Commit message: Bump pcb and can_controller
Parts:
- added R1: 10k, Resistor_SMD:R_0805_2012Metric, symbol Device:R_Small
- added R2: 1k, Resistor_SMD:R_0805_2012Metric, symbol Device:R_Small
- added U1: TXB0108PW, Package_SO:TSSOP-20_4.4x6.5mm_P0.65mm, symbol Logic_LevelTranslator:TXB0108PW
Connections:
- net +3V3: now also R2.2, U1.2 (V_{CCA})
- net GND: now also R1.1, U1.11 (GND)
- net SPI_CLK: now reaches U102.12 (SPI_CLK)
- net SPI_CLK: now also U1.20 (B1)
- net SPI_SDA1: now reaches U102.14 (SPI_SDA1/SPI_SDI)
- net SPI_SDA1: now also U1.18 (B2)
- net SPI_SDA2: now reaches U102.16 (SPI_SDA2)
- net SPI_SDA2: now also U1.17 (B3)
- net SPI_SDO: now reaches U102.17 (SPI_SD0)
- net SPI_SDO: now also U1.14 (B6)
- net SPI_SDA3: now reaches U102.18 (SPI_SDA3)
- net SPI_SDA3: now also U1.16 (B4)
- net SPI_SDA4: now reaches U102.20 (SPI_SDA4)
- net SPI_SDA4: now also U1.15 (B5)
- new net: R1.2, R2.1, U1.10 (OE)
- new net +5V: U1.19 (V_{CCB})
- no-connect marks 5 -> 2
Other:
- removed sheet MCU
- moved on the sheet: U102
